File: udayworks60.brd (EAGLE design)
At the start: 284.7 x 94.2 mm, 253 parts, among them J1 10137061-00021LF, SW1 SWITCH-SMD-EVP-BB2A9B00, X1 B4B-PH-SM4-TB, Y1 16MHz

Commit message: Initial Commit
Parts:
- removed D30: (no value), Components:SOD-123
- removed J1: 10137061-00021LF, 10137061-00021LF:AMPHENOL_10137061-00021LF
- removed R62, R74: 1K, Components:R0603
- added J2: TYPE-C-31-M-12, TYPE-C-31-M-12:HRO_TYPE-C-31-M-12
- moved D45 38.2 mm to (293.0, 95.1)
- moved FB2 13.2 mm to (22.0, 96.9), turned to 270 degrees
- moved R1 1.50 mm to (26.2, 94.9)
- moved R48 1.03 mm to (281.6, 51.5), turned to 180 degrees
- moved R2 0.35 mm to (28.6, 93.9), turned to 180 degrees
- renumbered SOMETHINGELSE to DELETE
Connections:
- removed net N$108: BACKSLASH.LED-, R35.2
- removed net N$111: NORMALSHIFT.LED-, R62.2
- removed net N$142: ENTER.LED-, R48.2
- removed net N$167: J1.A5, R1.1
- removed net N$168: J1.B5, R2.2
- removed net N$27: BACKSLASH.MX1, D29.A
- removed net N$77 (its old number): FB2.1, J1.S1, J1.S2, J1.S3, J1.S4
- new net N$145: J2.A5, R1.1
- new net N$147: J2.B5, R2.2
- new net N$59: DELETE.LED-, R48.2
- net C12: now also NORMALSHIFT.MX2
- net C13: no longer NORMALSHIFT.MX2
- net C4: now also U$1.26; no longer U$1.12
- net D+: now also J2.A6, J2.B6; no longer J1.A6, J1.B6
- net D-: now also J2.A7, J2.B7; no longer J1.A7, J1.B7
- net GND: now also J2.A1B12, J2.B1A12; no longer J1.A1, J1.A12, TP1.TP, TP2.TP, TP3.TP, TP4.TP, TP5.TP, TP6.TP
- net LEDS: no longer R62.1, R74.1
- net N$107: now also BACKSLASH.LED-, R35.2; no longer R74.2
- net N$112: now also NORMALSHIFT.LED-
- net N$127: now also ALT_R.LED-
- net N$143: now also ENTER.LED-; no longer DELETE.LED-
- net N$55: no longer ALT_R.MX1
- net N$58: now also ENTER.MX1
- net N$64: now also BACKSLASH.MX1, D29.A; no longer D30.A, ENTER.MX1
- net N$66: now also ALT_R.MX1
- net N$72: now also FB2.1, J2.S1, J2.S2, J2.S3, J2.S4; no longer J1.B1, J1.B12
- net N$83: now also U$1.29; no longer U$1.26
- net R2: no longer D30.C
- net R3: now also U$1.12; no longer D44.C, U$1.29
- net R4: now also D44.C
- net VBUS: now also J2.A4B9, J2.B4A9; no longer J1.A4, J1.A9, J1.B4, J1.B9
Routing:
- net GND: track 811.8 -> 673.4 mm, vias 16 -> 11
- net N$143: track 68.0 -> 12.9 mm, vias 1 -> 0
- net N$59: track 0.00 -> 47.6 mm, vias 0 -> 2
- net N$77: track 47.2 -> 11.6 mm, vias 1 -> 0
- net N$77 (its old number): track 24.8 -> 0.00 mm, vias 1 -> 0
- net R4: track 318.6 -> 343.4 mm, vias 2 -> 4
- net R3: track 322.7 -> 346.2 mm, vias 2 -> 4
- net N$168: track 19.9 -> 0.00 mm
- net N$66: track 3.71 -> 23.0 mm
- net VCC: track 2055.8 -> 2074.9 mm, vias 19 -> 21
- net N$55: track 24.6 -> 6.09 mm
- net C4: track 142.8 -> 158.9 mm, vias 1 -> 3
- net N$107: track 3.80 -> 18.4 mm
- net N$127: track 6.63 -> 20.6 mm
- net N$58: track 3.71 -> 15.7 mm
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