File: udayworks60.sch (EAGLE design)
At the start: 253 parts, among them J1 10137061-00021LF, SW1 SWITCH-SMD-EVP-BB2A9B00, X1 B4B-PH-SM4-TB, Y1 16MHz

Commit message: Initial Commit
Parts:
- removed D30: (no value), Components:DIODE-SOD-123
- removed J1: 10137061-00021LF, 10137061-00021LF:10137061-00021LF
- removed R62, R74: 1K, Components:RESISTOR-0603
- removed SOMETHINGELSE: KEYSWITCH-LED-MX-1U-LED, Keyboard:KEYSWITCH-LED-MX-1U-LED
- added DELETE: KEYSWITCH-LED-MX-1U-LED, Keyboard:KEYSWITCH-LED-MX-1U-LED
- added J2: TYPE-C-31-M-12, TYPE-C-31-M-12:TYPE-C-31-M-12
Connections:
- removed net N$108: BACKSLASH.LED-, R35.2
- removed net N$111: NORMALSHIFT.LED-, R62.2
- removed net N$142: ENTER.LED-, R48.2
- removed net N$167: J1.CC1, R1.1
- removed net N$168: J1.CC2, R2.2
- removed net N$27: BACKSLASH.P0, D29.A
- new net N$145: J2.CC1, R1.1
- new net N$147: J2.CC2, R2.2
- net C12: now also NORMALSHIFT.P1
- net C13: now also DELETE.P1; no longer NORMALSHIFT.P1, SOMETHINGELSE.P1
- net C4: now also U$1.PD6(T1/ADC9/!OC4D); no longer U$1.PB7(PCINT7/OC0A/OC1C/!RTS)
- net D+: now also J2.DP1, J2.DP2; no longer J1.DP1, J1.DP2
- net D-: now also J2.DN1, J2.DN2; no longer J1.DN1, J1.DN2
- net GND: now also J2.GND; no longer J1.GND_A1, J1.GND_A12, TP1.TP, TP2.TP, TP3.TP, TP4.TP, TP5.TP, TP6.TP
- net LEDS: no longer R62.1, R74.1
- net N$107: now also BACKSLASH.LED-, R35.2; no longer R74.2
- net N$112: now also NORMALSHIFT.LED-
- net N$127: now also ALT_R.LED-
- net N$143: now also ENTER.LED-; no longer SOMETHINGELSE.LED-
- net N$55: no longer ALT_R.P0
- net N$58: now also ENTER.P0
- net N$59: now also DELETE.LED-, R48.2; no longer D45.A, SOMETHINGELSE.P0
- net N$64: now also BACKSLASH.P0, D29.A; no longer D30.A, ENTER.P0
- net N$66: now also ALT_R.P0
- net N$72: now also FB2.1, J2.SHIELD; no longer J1.GND_B1, J1.GND_B12
- net N$77: now also D45.A, DELETE.P0; no longer FB2.1, J1.SHIELD
- net N$83: now also U$1.PB5(PCINT5/OC1A/ADC12/!OC4B); no longer U$1.PD6(T1/ADC9/!OC4D)
- net R2: no longer D30.C
- net R3: now also U$1.PB7(PCINT7/OC0A/OC1C/!RTS); no longer D44.C, U$1.PB5(PCINT5/OC1A/ADC12/!OC4B)
- net R4: now also D44.C
- net VBUS: now also J2.VBUS; no longer J1.VBUS_A4, J1.VBUS_A9, J1.VBUS_B4, J1.VBUS_B9
- net VCC: now also DELETE.LED+; no longer SOMETHINGELSE.LED+
Other:
- moved on the sheet: BACKSLASH2, D15, D44, D45, ENTER, FB2, ISOENTER, NORMALSHIFT, R1, R2, R49, R70
